Commit message: Small updates

File: my_car_description/urdf/gazebo_properties.urdf.xacro (robot description, xacro)
@@ -25,5 +25,5 @@
     <!-- Differential Drive Controller Plugin -->
     <gazebo>
-        <plugin name="diff_drive_controller" filename="libgazebo_ros_diff_drive.so">
+        <plugin name="back_diff_drive_controller" filename="libgazebo_ros_diff_drive.so">
             <ros>
                 <namespace>/</namespace>
@@ -34,4 +34,29 @@
             <left_joint>base_to_back_left_wheel_joint</left_joint>
             <right_joint>base_to_back_right_wheel_joint</right_joint>
+            <wheel_separation>0.4</wheel_separation>
+            <wheel_diameter>0.2</wheel_diameter>
+            <max_wheel_torque>20</max_wheel_torque>
+            <max_wheel_acceleration>1.0</max_wheel_acceleration>
+            <command_topic>cmd_vel</command_topic>
+            <publish_odom>true</publish_odom>
+            <publish_odom_tf>true</publish_odom_tf>
+            <publish_wheel_tf>true</publish_wheel_tf>
+            <odometry_topic>odom</odometry_topic>
+            <odometry_frame>odom</odometry_frame>
+            <robot_base_frame>base_footprint_link</robot_base_frame>
+            <pose_covariance_diagonal>0.0001 0.0001 0.0001 0.0 0.0 0.001</pose_covariance_diagonal>
+            <twist_covariance_diagonal>0.0001 0.0001 0.0001 0.0 0.0 0.001</twist_covariance_diagonal>
+        </plugin>
+    </gazebo>
+    <gazebo>
+        <plugin name="front_diff_drive_controller" filename="libgazebo_ros_diff_drive.so">
+            <ros>
+                <namespace>/</namespace>
+                <remapping>cmd_vel:=cmd_vel</remapping>
+                <remapping>odom:=odom</remapping>
+              </ros>
+            <update_rate>50</update_rate>
+            <left_joint>base_to_front_left_wheel_joint</left_joint>
+            <right_joint>base_to_front_right_wheel_joint</right_joint>
             <wheel_separation>0.4</wheel_separation>
             <wheel_diameter>0.2</wheel_diameter>

File: my_car_description/urdf/my_car.urdf.xacro (robot description, xacro)
@@ -61,4 +61,6 @@
     <xacro:wheel_link where="back" prefix="left"/>
     <xacro:wheel_link where="back" prefix="right"/>
+    <xacro:wheel_link where="front" prefix="left"/>
+    <xacro:wheel_link where="front" prefix="right"/>
     <link name="front_wheel_link">
         <visual>
@@ -103,4 +105,16 @@
         <axis xyz="0 1 0"/>
     </joint>
+    <joint name="base_to_front_right_wheel_joint" type="continuous">
+        <parent link="base_link"/>
+        <child link="front_right_wheel_link"/>
+        <origin xyz="0.15 -${(base_width/2) + (wheel_length/2)} 0" rpy="0 0 0"/>
+        <axis xyz="0 1 0"/>
+    </joint>
+    <joint name="base_to_front_left_wheel_joint" type="continuous">
+        <parent link="base_link"/>
+        <child link="front_left_wheel_link"/>
+        <origin xyz="0.15 ${(base_width/2) + (wheel_length/2)} 0" rpy="0 0 0"/>
+        <axis xyz="0 1 0"/>
+    </joint>
     <!-- Front caster wheel -->
     <joint name="base_to_front_wheel_joint" type="fixed">

Commit message: quick changes

File: my_car_description/urdf/gazebo_properties.urdf.xacro (robot description, xacro)
@@ -74,39 +74,3 @@
         </plugin>
     </gazebo>
-    <!-- Lidar Sensor Plugin -->
-    <gazebo reference="lidar_link">
-        <sensor type="ray" name="lidar_sensor">
-            <pose>0 0 0 0 0 0</pose>
-            <visualize>true</visualize>
-            <update_rate>10</update_rate>
-            <ray>
-                <scan>
-                    <horizontal>
-                        <samples>360</samples>
-                        <resolution>1</resolution>
-                        <min_angle>-3.14159</min_angle>
-                        <max_angle>3.14159</max_angle>
-                    </horizontal>
-                </scan>
-                <range>
-                    <min>0.5</min>
-                    <max>10.0</max>
-                    <resolution>0.01</resolution>
-                </range>
-                <noise>
-                    <type>gaussian</type>
-                    <mean>0.0</mean>
-                    <stddev>0.01</stddev>
-                </noise>
-            </ray>
-            <plugin name="gazebo_ros_lidar_controller" filename="libgazebo_ros_ray_sensor.so">
-                <ros>
-                    <namespace>/</namespace>
-                    <remapping>~/out:=scan</remapping>
-                </ros>
-                <output_type>sensor_msgs/LaserScan</output_type>
-                <frame_name>lidar_link</frame_name>
-            </plugin>
-        </sensor>
-    </gazebo>
 </robot>

File: my_car_description/urdf/my_car.urdf.xacro (robot description, xacro)
@@ -3,123 +3,6 @@
     <xacro:include filename="common_properties.urdf.xacro"/>
     <xacro:include filename="gazebo_properties.urdf.xacro"/>
-    <xacro:property name="base_length" value="0.6"/>
-    <xacro:property name="base_width" value="0.4"/>
-    <xacro:property name="base_height" value="0.2"/>
-    <xacro:property name="wheel_radius" value="0.1"/>
-    <xacro:property name="wheel_length" value="0.1"/>
-    <xacro:macro name="wheel_link" params="where prefix">
-        <link name="${where}_${prefix}_wheel_link">
-            <visual>
-                <geometry>
-                    <cylinder radius="${wheel_radius}" length="${wheel_length}"/>
-                </geometry>
-                <origin xyz="0 0 0" rpy="${pi/2} 0 0"/>
-                <material name="yellow"/>
-            </visual>
-            <collision>
-                <geometry>
-                    <cylinder radius="${wheel_radius}" length="${wheel_length}"/>
-                </geometry>
-                <origin xyz="0 0 0" rpy="${pi/2} 0 0"/>
-            </collision>
-            <xacro:wheel_inertia r="${wheel_radius}" h="${wheel_length}" m="5.0" xyz="0 0 0" rpy="${pi/2} 0 0" />
-        </link>
-    </xacro:macro>
-    <link name="base_footprint_link"/>
-    <link name="base_link">
-        <visual>
-            <geometry>
-                <box size="${base_length} ${base_width} ${base_height}"/>
-            </geometry>
-            <origin xyz="0 0 0.1" rpy="0 0 0"/>
-            <material name="blue"/>
-        </visual>
-        <collision>
-            <geometry>
-                <box size="${base_length} ${base_width} ${base_height}"/>
-            </geometry>
-            <origin xyz="0 0 0.1" rpy="0 0 0"/>
-        </collision>
-        <xacro:box_inertia l="${base_length}" w="${base_width}" h="${base_height}" m="35" xyz="0 0 0.1" rpy="0 0 0"/>
-    </link>
-    <link name="lidar_link">
-        <visual>
-            <geometry>
-                <cylinder radius="0.1" length="0.2"/>
-            </geometry>
-            <origin xyz="0 0 0.1" rpy="0 0 0"/>
-            <material name="green"/>
-        </visual>
-        <collision>
-            <geometry>
-                <cylinder radius="0.1" length="0.2"/>
-            </geometry>
-            <origin xyz="0 0 0.1" rpy="0 0 0"/>
-        </collision>
-        <xacro:wheel_inertia r="0.1" h="0.2" m="4.0" xyz="0 0 0.1" rpy="0 0 0" />
-    </link>
-    <xacro:wheel_link where="back" prefix="left"/>
-    <xacro:wheel_link where="back" prefix="right"/>
-    <xacro:wheel_link where="front" prefix="left"/>
-    <xacro:wheel_link where="front" prefix="right"/>
-    <link name="front_wheel_link">
-        <visual>
-            <geometry>
-                <sphere radius="0.05"/>
-            </geometry>
-            <origin xyz="0 0 0" rpy="0 0 0"/>
-            <material name="black"/>
-        </visual>
-        <collision>
-            <geometry>
-                <sphere radius="0.05"/>
-            </geometry>
-            <origin xyz="0 0 0" rpy="0 0 0"/>
-        </collision>
-        <xacro:sphere_inertia m="2.0" r="0.05" xyz="0 0 0" rpy="0 0 0" />
-    </link>
-    <!-- Include camera -->
+    <xacro:include filename="mobile_base.xacro"/>
+    <xacro:include filename="lidar.xacro"/>
     <xacro:include filename="camera.urdf.xacro"/>
-    <!-- JOINTS -->
-    <joint name="base_footprint_to_base" type="fixed">
-        <parent link="base_footprint_link"/>
-        <child link="base_link"/>
-        <origin xyz="0 0 ${wheel_radius}" rpy="0 0 0"/>
-    </joint>
-    <joint name="base_to_lidar_joint" type="fixed">
-        <parent link="base_link"/>
-        <child link="lidar_link"/>
-        <origin xyz="0 0 0.2" rpy="0 0 0"/>
-    </joint>
-    <!-- Back wheels - these are the driving wheels -->
-    <joint name="base_to_back_right_wheel_joint" type="continuous">
-        <parent link="base_link"/>
-        <child link="back_right_wheel_link"/>
-        <origin xyz="-0.15 -${(base_width/2) + (wheel_length/2)} 0" rpy="0 0 0"/>
-        <axis xyz="0 1 0"/>
-    </joint>
-    <joint name="base_to_back_left_wheel_joint" type="continuous">
-        <parent link="base_link"/>
-        <child link="back_left_wheel_link"/>
-        <origin xyz="-0.15 ${(base_width/2) + (wheel_length/2)} 0" rpy="0 0 0"/>
-        <axis xyz="0 1 0"/>
-    </joint>
-    <joint name="base_to_front_right_wheel_joint" type="continuous">
-        <parent link="base_link"/>
-        <child link="front_right_wheel_link"/>
-        <origin xyz="0.15 -${(base_width/2) + (wheel_length/2)} 0" rpy="0 0 0"/>
-        <axis xyz="0 1 0"/>
-    </joint>
-    <joint name="base_to_front_left_wheel_joint" type="continuous">
-        <parent link="base_link"/>
-        <child link="front_left_wheel_link"/>
-        <origin xyz="0.15 ${(base_width/2) + (wheel_length/2)} 0" rpy="0 0 0"/>
-        <axis xyz="0 1 0"/>
-    </joint>
-    <!-- Front caster wheel -->
-    <joint name="base_to_front_wheel_joint" type="fixed">
-        <parent link="base_link"/>
-        <child link="front_wheel_link"/>
-        <origin xyz="${base_length/2 - 0.05} 0 -${wheel_radius/2}" rpy="0 0 0"/>
-    </joint>
 </robot>
