Commit message: base_link perspective_shift

File: my_car_description/urdf/camera.urdf.xacro (robot description, xacro)
@@ -18,5 +18,5 @@
     </link>
     <joint name="base_to_camera_joint" type="fixed">
-        <parent link="base_link"/>
+        <parent link="main_link"/>
         <child link="camera_link"/>
         <origin xyz="${base_length/2.0} 0 ${base_height}" rpy="0 0 0"/>

File: my_car_description/urdf/gazebo_properties.urdf.xacro (robot description, xacro)
@@ -2,5 +2,5 @@
 <robot xmlns:xacro="http://www.ros.org/wiki/xacro">
     <!-- Gazebo materials for visual links -->
-    <gazebo reference="base_link">
+    <gazebo reference="main_link">
         <material>Gazebo/Blue</material>
     </gazebo>
@@ -44,5 +44,5 @@
             <odometry_topic>odom</odometry_topic>
             <odometry_frame>odom</odometry_frame>
-            <robot_base_frame>base_footprint_link</robot_base_frame>
+            <robot_base_frame>base_link</robot_base_frame>
             <pose_covariance_diagonal>0.0001 0.0001 0.0001 0.0 0.0 0.001</pose_covariance_diagonal>
             <twist_covariance_diagonal>0.0001 0.0001 0.0001 0.0 0.0 0.001</twist_covariance_diagonal>
@@ -69,5 +69,5 @@
             <odometry_topic>odom</odometry_topic>
             <odometry_frame>odom</odometry_frame>
-            <robot_base_frame>base_footprint_link</robot_base_frame>
+            <robot_base_frame>base_link</robot_base_frame>
             <pose_covariance_diagonal>0.0001 0.0001 0.0001 0.0 0.0 0.001</pose_covariance_diagonal>
             <twist_covariance_diagonal>0.0001 0.0001 0.0001 0.0 0.0 0.001</twist_covariance_diagonal>

File: my_car_description/urdf/lidar.xacro (robot description, xacro)
@@ -18,5 +18,5 @@
     </link>
     <joint name="base_to_lidar_joint" type="fixed">
-        <parent link="base_link"/>
+        <parent link="main_link"/>
         <child link="lidar_link"/>
         <origin xyz="0 0 0.2" rpy="0 0 0"/>

File: my_car_description/urdf/mobile_base.xacro (robot description, xacro)
@@ -24,6 +24,6 @@
         </link>
     </xacro:macro>
-    <link name="base_footprint_link"/>
-    <link name="base_link">
+    <link name="base_link"/>
+    <link name="main_link">
         <visual>
             <geometry>
@@ -63,11 +63,11 @@
     <!-- JOINTS -->
     <joint name="base_footprint_to_base" type="fixed">
-        <parent link="base_footprint_link"/>
-        <child link="base_link"/>
+        <parent link="base_link"/>
+        <child link="main_link"/>
         <origin xyz="0 0 ${wheel_radius}" rpy="0 0 0"/>
     </joint>
     <!-- Back wheels - these are the driving wheels -->
     <joint name="base_to_back_right_wheel_joint" type="continuous">
-        <parent link="base_link"/>
+        <parent link="main_link"/>
         <child link="back_right_wheel_link"/>
         <origin xyz="-0.15 -${(base_width/2) + (wheel_length/2)} 0" rpy="0 0 0"/>
@@ -75,5 +75,5 @@
     </joint>
     <joint name="base_to_back_left_wheel_joint" type="continuous">
-        <parent link="base_link"/>
+        <parent link="main_link"/>
         <child link="back_left_wheel_link"/>
         <origin xyz="-0.15 ${(base_width/2) + (wheel_length/2)} 0" rpy="0 0 0"/>
@@ -81,5 +81,5 @@
     </joint>
     <joint name="base_to_front_right_wheel_joint" type="continuous">
-        <parent link="base_link"/>
+        <parent link="main_link"/>
         <child link="front_right_wheel_link"/>
         <origin xyz="0.15 -${(base_width/2) + (wheel_length/2)} 0" rpy="0 0 0"/>
@@ -87,5 +87,5 @@
     </joint>
     <joint name="base_to_front_left_wheel_joint" type="continuous">
-        <parent link="base_link"/>
+        <parent link="main_link"/>
         <child link="front_left_wheel_link"/>
         <origin xyz="0.15 ${(base_width/2) + (wheel_length/2)} 0" rpy="0 0 0"/>
@@ -94,5 +94,5 @@
     <!-- Front caster wheel -->
     <joint name="base_to_front_wheel_joint" type="fixed">
-        <parent link="base_link"/>
+        <parent link="main_link"/>
         <child link="front_wheel_link"/>
         <origin xyz="${base_length/2 - 0.05} 0 -${wheel_radius/2}" rpy="0 0 0"/>

File: my_car_description/urdf/my_car.urdf.xacro (robot description, xacro)
@@ -6,3 +6,4 @@
     <xacro:include filename="lidar.xacro"/>
     <xacro:include filename="camera.urdf.xacro"/>
+    <xacro:include filename="my_car_control.urdf.xacro"/>
 </robot>
