Commit message: minor changes

File: my_car_description/urdf/common_properties.urdf.xacro (robot description, xacro)
@@ -9,4 +9,7 @@
     <material name="red">
         <color rgba="1 0 0 1"/>
+    </material>
+    <material name="yellow">
+        <color rgba="1 1 0 1"/>
     </material>
     <material name="black">

File: my_car_description/urdf/gazebo_properties.urdf.xacro (robot description, xacro)
@@ -6,14 +6,14 @@
     </gazebo>
     <gazebo reference="back_right_wheel_link">
-        <material>Gazebo/Black</material>
+        <material>Gazebo/Yellow</material>
     </gazebo>
     <gazebo reference="back_left_wheel_link">
-        <material>Gazebo/Black</material>
+        <material>Gazebo/Yellow</material>
     </gazebo>
     <gazebo reference="front_right_wheel_link">
-        <material>Gazebo/Black</material>
+        <material>Gazebo/Yellow</material>
     </gazebo>
     <gazebo reference="front_left_wheel_link">
-        <material>Gazebo/Black</material>
+        <material>Gazebo/Yellow</material>
     </gazebo>
     <gazebo reference="camera_link">
@@ -21,5 +21,5 @@
     </gazebo>
     <gazebo reference="lidar_link">
-        <material>Gazebo/Red</material>
+        <material>Gazebo/Blue</material>
     </gazebo>
     <!-- Differential Drive Controller Plugin -->

File: my_car_description/urdf/my_car.urdf.xacro (robot description, xacro)
@@ -15,5 +15,5 @@
                 </geometry>
                 <origin xyz="0 0 0" rpy="${pi/2} 0 0"/>
-                <material name="black"/>
+                <material name="yellow"/>
             </visual>
             <collision>

Commit message: screen update

File: my_car_description/urdf/common_properties.urdf.xacro (robot description, xacro)
@@ -3,4 +3,7 @@
     <material name="blue">
         <color rgba="0 0 1 1"/>
+    </material>
+    <material name="orange">
+        <color rgba="1 0.5 0 1"/>
     </material>
     <material name="green">

File: my_car_description/urdf/gazebo_properties.urdf.xacro (robot description, xacro)
@@ -3,5 +3,5 @@
     <!-- Gazebo materials for visual links -->
     <gazebo reference="main_link">
-        <material>Gazebo/Blue</material>
+        <material>Gazebo/Orange</material>
     </gazebo>
     <gazebo reference="back_right_wheel_link">

File: my_car_description/urdf/lidar.xacro (robot description, xacro)
@@ -7,5 +7,5 @@
             </geometry>
             <origin xyz="0 0 0.1" rpy="0 0 0"/>
-            <material name="green"/>
+            <material name="blue"/>
         </visual>
         <collision>

File: my_car_description/urdf/mobile_base.xacro (robot description, xacro)
@@ -31,5 +31,5 @@
             </geometry>
             <origin xyz="0 0 0.1" rpy="0 0 0"/>
-            <material name="blue"/>
+            <material name="orange"/>
         </visual>
         <collision>
